Commit message: add baxter_kinect.urdf

File: baxter_description/urdf/baxter_kinect.urdf (robot description, URDF)
Before this commit: robot baxter, 49 links, 48 joints
Links:
- added link xtion_depth_frame
- added link xtion_depth_optical_frame
- added link xtion_link, mass 0.200
- added link xtion_rgb_frame
- added link xtion_rgb_optical_frame
Joints:
- added joint xtion_depth_joint: type fixed, parent xtion_link, child xtion_depth_frame, origin xyz=0.0 0.049 0.0 rpy=0 0 0
- added joint xtion_depth_optical_joint: type fixed, parent xtion_depth_frame, child xtion_depth_optical_frame, origin xyz=0 0 0 rpy=-1.57079632679 0.0 -1.57079632679
- added joint xtion_joint: type fixed, parent head, child xtion_link, origin xyz=-0.069 0.0 0.263 rpy=0 0 0
- added joint xtion_rgb_joint: type fixed, parent xtion_link, child xtion_rgb_frame, origin xyz=0.0 0.022 0.0 rpy=0 0 0
- added joint xtion_rgb_optical_joint: type fixed, parent xtion_rgb_frame, child xtion_rgb_optical_frame, origin xyz=0 0 0 rpy=-1.57079632679 0.0 -1.57079632679
