Commit message: use smaller collision head

File: baxter_description/urdf/baxter_base/baxter_base.urdf.xacro (robot description, xacro)
@@ -153,5 +153,5 @@
       <origin rpy="0 0 0.0" xyz="-0.07 -0.04 0.0"/>
       <geometry>
-        <sphere radius="0.22"/>
+        <sphere radius="0.1"/>
       </geometry>
     </collision>
@@ -175,5 +175,5 @@
       <origin rpy="0 0 0" xyz="-0.07 0.04 0.00"/>
       <geometry>
-        <sphere radius="0.22"/>
+        <sphere radius="0.1"/>
       </geometry>
     </collision>
